Commit message: tilting quad

File: urdf/ndt2/ndt2.xacro (robot description, xacro)
@@ -31,5 +31,5 @@
   <xacro:property name="rotor_offset_top" value="0.01" /> <!-- [m] -->
   <xacro:property name="radius_rotor" value="0.1" /> <!-- [m] -->
-  <xacro:property name="motor_constant" value="0.00019065" /> <!-- [kg.m/s^2] -->
+  <xacro:property name="motor_constant" value="0.00190650" /> <!-- [kg.m/s^2] -->
   <xacro:property name="moment_constant" value="0.000001333" /> <!-- 0.06 [m] -->
   <xacro:property name="time_constant_up" value="0.0125" /> <!-- [s] -->
@@ -40,5 +40,5 @@
 	<xacro:property name="x_rotor" value="0.121"  />
 	<xacro:property name="y_rotor" value="0.121"  />
-	<xacro:property name="z_rotor" value="0.075"  />
+	<xacro:property name="z_rotor" value="0.035"  />
 	<xacro:include filename="$(find mav_description)/urdf/ndt2/ndt2.trans" />
 	<xacro:include filename="$(find mav_description)/urdf/ndt2/ndt2.gazebo" />
@@ -98,5 +98,5 @@
     </visual>
     <collision>
-      <origin rpy="0 0 0" xyz="-0.16832475 0.175539 -0.02"/>
+      <origin rpy="0 0 3.1415" xyz="0.0 0.0 -0.02"/>
       <geometry>
         <mesh filename="$(find mav_description)/meshes/ndt2/arm_4.stl"/>
@@ -105,5 +105,6 @@
   </link>
    <joint name="tilt_motor_4" type="revolute">
-    <origin rpy="0 0 3.1415" xyz="0.16832475 -0.175539 0.04"/>
+    <!--<origin rpy="0 0 3.1415" xyz="0.16832475 -0.175539 0.04"/>-->
+    <origin rpy="0 0 3.1415" xyz="0.0 0.0 0.02"/>
     <parent link="base_link"/>
     <child link="arm_4"/>
@@ -118,5 +119,6 @@
     </inertial>
     <visual>
-      <origin rpy="0 0 0" xyz="0.224433 -0.234052 -0.04"/>
+      <!--<origin rpy="0 0 0" xyz="0.224433 -0.234052 -0.04"/>-->
+      <origin rpy="0 0 0" xyz="0.0 -0.0 -0.02"/>
       <geometry>
         <mesh filename="$(find mav_description)/meshes/ndt2/arm_2.stl"/>
@@ -124,5 +126,5 @@
     </visual>
     <collision>
-      <origin rpy="0 0 0" xyz="0.224433 -0.234052 -0.04"/>
+      <origin rpy="0 0 0" xyz="0.0 -0.0 -0.02"/>
       <geometry>
         <mesh filename="$(find mav_description)/meshes/ndt2/arm_2.stl"/>
@@ -131,5 +133,6 @@
   </link>
   <joint name="tilt_motor_2" type="revolute">
-    <origin rpy="0 0 0" xyz="-0.224433 0.234052 0.04"/>
+    <!--<origin rpy="0 0 0" xyz="-0.224433 0.234052 0.04"/>-->
+    <origin rpy="0 0 0" xyz="-0.0 0.0 0.02"/>
     <parent link="base_link"/>
     <child link="arm_2"/>
@@ -144,5 +147,5 @@
     </inertial>
     <visual>
-      <origin rpy="0 0 0" xyz="0.224433 0.234052 -0.04"/>
+      <origin rpy="0 0 3.1415" xyz="0.0 0.0 -0.02"/>
       <geometry>
         <mesh filename="$(find mav_description)/meshes/ndt2/arm_3.stl"/>
@@ -150,5 +153,5 @@
     </visual>
     <collision>
-      <origin rpy="0 0 0" xyz="0.224433 0.234052 -0.04"/>
+      <origin rpy="0 0 3.1415" xyz="0.0 0.0 -0.02"/>
       <geometry>
         <mesh filename="$(find mav_description)/meshes/ndt2/arm_3.stl"/>
@@ -157,5 +160,5 @@
   </link>
    <joint name="tilt_motor_3" type="revolute">
-    <origin rpy="0 0 0" xyz="-0.224433 -0.234052 0.04"/>
+    <origin rpy="0 0 3.1415" xyz="0.0 0.0 0.02"/>
     <parent link="base_link"/>
     <child link="arm_3"/>
@@ -170,5 +173,5 @@
     </inertial>
     <visual>
-      <origin rpy="0 0 0" xyz="-0.224433 -0.234052 -0.04"/>
+      <origin rpy="0 0 3.1415" xyz="0.0 0.0 -0.02"/>
       <geometry>
         <mesh filename="$(find mav_description)/meshes/ndt2/arm_1.stl"/>
@@ -176,5 +179,5 @@
     </visual>
     <collision>
-      <origin rpy="0 0 0" xyz="-0.224433 -0.234052 -0.04"/>
+      <origin rpy="0 0 3.1415" xyz="0.0 0.0 -0.02"/>
       <geometry>
         <mesh filename="$(find mav_description)/meshes/ndt2/arm_1.stl"/>
@@ -183,5 +186,5 @@
   </link>
  <joint name="tilt_motor_1" type="revolute">
-    <origin rpy="0 0 0" xyz="0.224433 0.234052 0.04"/>
+    <origin rpy="0 0 3.1415" xyz="0.0 0.0 0.02"/>
     <parent link="base_link"/>
     <child link="arm_1"/>
@@ -207,5 +210,6 @@
     color="Red"
     mesh="ndt2/prop.stl">
-    <origin xyz="${x_rotor} -${y_rotor} ${z_rotor}" rpy="0 0 0" />
+    <!--<origin xyz="${x_rotor} -${y_rotor} ${z_rotor}" rpy="0 0 0" />-->
+    <origin xyz="-0.175 0.175 ${z_rotor}" rpy="0 0 0" />
     <xacro:insert_block name="rotor_inertia" />
   </xacro:vertical_rotor>
@@ -228,5 +232,5 @@
     color="Blue"
     mesh="ndt2/prop.stl">
-    <origin xyz="-${x_rotor} ${y_rotor} ${z_rotor}" rpy="0 0 0" />
+    <origin xyz="-0.175 0.175 ${z_rotor}" rpy="0 0 0" />
     <xacro:insert_block name="rotor_inertia" />
   </xacro:vertical_rotor>
@@ -249,5 +253,5 @@
     color="Red"
     mesh="ndt2/prop.stl">
-    <origin xyz="${x_rotor} ${y_rotor} ${z_rotor}" rpy="0 0 0" />
+    <origin xyz="-0.175 -0.175 ${z_rotor}" rpy="0 0 0" />
     <xacro:insert_block name="rotor_inertia" />
   </xacro:vertical_rotor>
@@ -270,5 +274,5 @@
     color="Blue"
     mesh="ndt2/prop.stl">
-    <origin xyz="-${x_rotor} -${y_rotor} ${z_rotor}" rpy="0 0 0" />
+    <origin xyz="0.175 0.175 ${z_rotor}" rpy="0 0 0" />
     <xacro:insert_block name="rotor_inertia" />
   </xacro:vertical_rotor>

Commit message: new param for ndt2

File: urdf/ndt2/ndt2.xacro (robot description, xacro)
@@ -21,21 +21,34 @@
   <xacro:property name="mesh_scale_prop" value="1 1 1"/>
   <xacro:property name="mesh_file" value="ndt2/chassis_res.stl" />
-  <xacro:property name="mass" value="9.489" /> <!-- chassis mass [kg] -->
-  <xacro:property name="arm_mass" value="0.630" /> <!-- [kg] -->
+  <xacro:property name="mass" value="1.5" /> <!-- chassis mass [kg] -->
+  <xacro:property name="arm_mass" value="0.001" /> <!-- [kg] -->
   <xacro:property name="body_width" value="0.470" /> <!-- [m] -->
   <xacro:property name="body_height" value="0.380" /> <!-- [m] -->
-  <xacro:property name="mass_rotor" value="0.005" /> <!-- [kg] -->
+  <xacro:property name="mass_rotor" value="0.001" /> <!-- [kg] -->
   <xacro:property name="arm_length" value="0.17" /> <!-- [m] -->
   <xacro:property name="arm_width" value="0.340" /> <!-- [m] -->
   <xacro:property name="arm_height" value="0.06" /> <!-- [m] -->
   <xacro:property name="rotor_offset_top" value="0.01" /> <!-- [m] -->
-  <xacro:property name="radius_rotor" value="0.1" /> <!-- [m] -->
-  <xacro:property name="motor_constant" value="0.00190650" /> <!-- [kg.m/s^2] -->
-  <xacro:property name="moment_constant" value="0.000001333" /> <!-- 0.06 [m] -->
+ <!-- <xacro:property name="radius_rotor" value="0.1" />
+  <xacro:property name="motor_constant" value="0.0019065" />
+  <xacro:property name="moment_constant" value="0.000001333" />
+  <xacro:property name="time_constant_up" value="0.0125" />
+  <xacro:property name="time_constant_down" value="0.025" />
+  <xacro:property name="max_rot_velocity" value="5000" />
+  <xacro:property name="rotor_drag_coefficient" value="1.75e-04" />
+  <xacro:property name="rolling_moment_coefficient" value="0.000001" />
+-->
+ <xacro:property name="radius_rotor" value="0.128" /> <!-- [m] -->
+  <xacro:property name="motor_constant" value="8.54858e-06" /> <!-- [kg.m/s^2] -->
+  <xacro:property name="moment_constant" value="0.06" /> <!-- [m] -->
   <xacro:property name="time_constant_up" value="0.0125" /> <!-- [s] -->
   <xacro:property name="time_constant_down" value="0.025" /> <!-- [s] -->
-  <xacro:property name="max_rot_velocity" value="5000" /> <!-- [rad/s] -->
+  <xacro:property name="max_rot_velocity" value="1100" /> <!-- [rad/s] -->
+  <xacro:property name="sin30" value="0.5" />
+  <xacro:property name="cos30" value="0.866025403784" />
+  <xacro:property name="sqrt2" value="1.4142135623730951" />
   <xacro:property name="rotor_drag_coefficient" value="1.75e-04" />
   <xacro:property name="rolling_moment_coefficient" value="0.000001" />
+  <xacro:property name="color" value="$(arg visual_material)" />
 	<xacro:property name="x_rotor" value="0.121"  />
 	<xacro:property name="y_rotor" value="0.121"  />

Commit message: tilting quad added

File: urdf/ndt2/ndt2.xacro (robot description, xacro)
@@ -40,5 +40,5 @@
 -->
  <xacro:property name="radius_rotor" value="0.128" /> <!-- [m] -->
-  <xacro:property name="motor_constant" value="8.54858e-06" /> <!-- [kg.m/s^2] -->
+  <xacro:property name="motor_constant" value="8.54858e-05" /> <!-- [kg.m/s^2] -->
   <xacro:property name="moment_constant" value="0.06" /> <!-- [m] -->
   <xacro:property name="time_constant_up" value="0.0125" /> <!-- [s] -->

File: urdf/ndt2/ndt2_base.xacro (robot description, xacro)
@@ -15,4 +15,5 @@
   <xacro:include filename="$(find mav_description)/urdf/component_snippets.xacro" />
   <xacro:include filename="$(find mav_description)/urdf/ndt2/ndt2.xacro" />
+  <xacro:arg name="with_arm" default="false" />
   <xacro:ros_interface_macro
 	  namespace="${namespace}"
@@ -24,6 +25,7 @@
     </plugin>
   </gazebo>
-  <!--
-  <xacro:include filename="$(find Aerial_core_description)/urdf/Aerial_core.xacro" />
-  -->
+  <!---->
+  <xacro:if value="$(arg with_arm)">
+    <xacro:include filename="$(find aerial_arm_description)/urdf/Aerial_core.xacro" />
+  </xacro:if>
 </robot>
