Commit message: update

File: urdf/ndt2/ndt2 (copy).xacro (robot description, xacro)
@@ -21,6 +21,6 @@
   <xacro:property name="mesh_scale_prop" value="1 1 1"/>
   <xacro:property name="mesh_file" value="ndt2/chassis_res.stl" />
-  <xacro:property name="mass" value="5" /> <!-- chassis mass [kg] -->
-  <xacro:property name="arm_mass" value="0.1" /> <!-- [kg] -->
+  <xacro:property name="mass" value="1.5" /> <!-- chassis mass [kg] -->
+  <xacro:property name="arm_mass" value="0.001" /> <!-- [kg] -->
   <xacro:property name="body_width" value="0.470" /> <!-- [m] -->
   <xacro:property name="body_height" value="0.380" /> <!-- [m] -->
