Commit message: ft plugin for hexa_tilt

File: urdf/firefly_tilt/firefly_tilt_base.xacro (robot description, xacro)
@@ -12,3 +12,11 @@
     </plugin>
   </gazebo>
+	<gazebo>
+    <plugin filename="libforce_plugin.so" name="force">
+      <debug>1</debug>
+      <body_frame>1</body_frame>
+      <link_name>base_link</link_name>
+      <topic_name>/firefly_tilt/ft</topic_name>
+    </plugin>
+  </gazebo>
 </robot>

File: urdf/hummingbird/hummingbird.xacro (robot description, xacro)
@@ -154,89 +154,3 @@
     <xacro:insert_block name="rotor_inertia" />
   </xacro:vertical_rotor>
-  <!--
-  <xacro:vertical_rotor
-    robot_namespace="${namespace}"
-    suffix="front"
-    direction="cw"
-    motor_constant="${motor_constant}"
-    moment_constant="${moment_constant}"
-    parent="base_link"
-    mass_rotor="${mass_rotor}"
-    radius_rotor="${radius_rotor}"
-    time_constant_up="${time_constant_up}"
-    time_constant_down="${time_constant_down}"
-    max_rot_velocity="${max_rot_velocity}"
-    motor_number="0"
-    rotor_drag_coefficient="${rotor_drag_coefficient}"
-    rolling_moment_coefficient="${rolling_moment_coefficient}"
-    mesh="iris_prop"
-    mesh_scale="${mesh_scale_prop}"
-    color="Blue">
-    <origin xyz="${arm_length} 0 ${rotor_offset_top}" rpy="0 0 0" />
-    <xacro:insert_block name="rotor_inertia" />
-  </xacro:vertical_rotor>
-    <xacro:vertical_rotor
-    robot_namespace="${namespace}"
-    suffix="left"
-    direction="ccw"
-    motor_constant="${motor_constant}"
-    moment_constant="${moment_constant}"
-    parent="base_link"
-    mass_rotor="${mass_rotor}"
-    radius_rotor="${radius_rotor}"
-    time_constant_up="${time_constant_up}"
-    time_constant_down="${time_constant_down}"
-    max_rot_velocity="${max_rot_velocity}"
-    motor_number="1"
-    rotor_drag_coefficient="${rotor_drag_coefficient}"
-    rolling_moment_coefficient="${rolling_moment_coefficient}"
-    mesh="iris_prop"
-    mesh_scale="${mesh_scale_prop}"
-    color="Blue">
-    <origin xyz="0 ${arm_length} ${rotor_offset_top}" rpy="0 0 0" />
-    <xacro:insert_block name="rotor_inertia" />
-  </xacro:vertical_rotor>
-  <xacro:vertical_rotor
-    robot_namespace="${namespace}"
-    suffix="back"
-    direction="cw"
-    motor_constant="${motor_constant}"
-    moment_constant="${moment_constant}"
-    parent="base_link"
-    mass_rotor="${mass_rotor}"
-    radius_rotor="${radius_rotor}"
-    time_constant_up="${time_constant_up}"
-    time_constant_down="${time_constant_down}"
-    max_rot_velocity="${max_rot_velocity}"
-    motor_number="2"
-    rotor_drag_coefficient="${rotor_drag_coefficient}"
-    rolling_moment_coefficient="${rolling_moment_coefficient}"
-    mesh="iris_prop"
-    mesh_scale="${mesh_scale_prop}"
-    color="Blue">
-    <origin xyz="-${arm_length} 0 ${rotor_offset_top}" rpy="0 0 0" />
-    <xacro:insert_block name="rotor_inertia" />
-  </xacro:vertical_rotor>
-    <xacro:vertical_rotor
-    robot_namespace="${namespace}"
-    suffix="right"
-    direction="ccw"
-    motor_constant="${motor_constant}"
-    moment_constant="${moment_constant}"
-    parent="base_link"
-    mass_rotor="${mass_rotor}"
-    radius_rotor="${radius_rotor}"
-    time_constant_up="${time_constant_up}"
-    time_constant_down="${time_constant_down}"
-    max_rot_velocity="${max_rot_velocity}"
-    motor_number="3"
-    rotor_drag_coefficient="${rotor_drag_coefficient}"
-    rolling_moment_coefficient="${rolling_moment_coefficient}"
-    mesh="iris_prop"
-    mesh_scale="${mesh_scale_prop}"
-    color="Blue">
-    <origin xyz="0 -${arm_length} ${rotor_offset_top}" rpy="0 0 0" />
-    <xacro:insert_block name="rotor_inertia" />
-  </xacro:vertical_rotor>
-  -->
 </robot>

File: urdf/hummingbird/hummingbird_base.xacro (robot description, xacro)
@@ -38,3 +38,12 @@
 	  motor_size="4" >
 	</xacro:ros_interface_macro>
+<!---->
+  <gazebo>
+    <plugin filename="libforce_plugin.so" name="force">
+      <debug>1</debug>
+      <body_frame>1</body_frame>
+      <link_name>base_link</link_name>
+      <topic_name>/hummingbird/ft</topic_name>
+    </plugin>
+  </gazebo>
 </robot>
